File: Diseños/Circuito maquina garra peluches.sch (EAGLE design)
At the start: 7 parts, among them U1 ARDUINO_PRO_MINI

Commit message: avances documentación
Connections:
- net TXO renamed TXO1
- net RXI: now also MPU6050.8
- net VCC: no longer MPU6050.8
Changed lines of the file:
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@@
 <label x="101.6" y="50.8" size="1.778" layer="95"/>
-</segment>
-<segment>
-<pinref part="MPU6050" gate="1" pin="8"/>
-<wire x1="10.16" y1="66.04" x2="17.78" y2="66.04" width="0.1524" layer="91"/>
-<label x="12.7" y="66.04" size="1.778" layer="95"/>
 </segment>
 </net>
@@
 </segment>
 </net>
-<net name="TXO" class="0">
-<segment>
-<wire x1="114.3" y1="55.88" x2="101.6" y2="55.88" width="0.1524" layer="91"/>
-<pinref part="PROG" gate="A" pin="2"/>
-<label x="101.6" y="55.88" size="1.778" layer="95"/>
-</segment>
-<segment>
-<pinref part="U1" gate="G$1" pin="TXO"/>
-<wire x1="73.66" y1="68.58" x2="81.28" y2="68.58" width="0.1524" layer="91"/>
-<label x="78.74" y="68.58" size="1.778" layer="95"/>
-</segment>
-</net>
 <net name="RXI" class="0">
 <segment>
@@
 <wire x1="73.66" y1="66.04" x2="81.28" y2="66.04" width="0.1524" layer="91"/>
 <label x="78.74" y="66.04" size="1.778" layer="95"/>
+</segment>
+<segment>
+<pinref part="MPU6050" gate="1" pin="8"/>
+<wire x1="10.16" y1="66.04" x2="20.32" y2="66.04" width="0.1524" layer="91"/>
+<label x="12.7" y="66.04" size="1.778" layer="95"/>
+<wire x1="20.32" y1="66.04" x2="20.32" y2="73.66" width="0.1524" layer="91"/>
 </segment>
 </net>
@@
 </segment>
 </net>
+<net name="TXO1" class="0">
+<segment>
+<pinref part="U1" gate="G$1" pin="TXO"/>
+<wire x1="73.66" y1="68.58" x2="81.28" y2="68.58" width="0.1524" layer="91"/>
+<label x="78.74" y="68.58" size="1.778" layer="95"/>
+</segment>
+<segment>
+<wire x1="114.3" y1="55.88" x2="101.6" y2="55.88" width="0.1524" layer="91"/>
+<pinref part="PROG" gate="A" pin="2"/>
+<label x="101.6" y="55.88" size="1.778" layer="95"/>
+</segment>
+</net>
